Commit message: docs & cad: integrate 3D CAD models, FEA analysis, automated launch, and comprehensive presentation
- Add master SolidWorks assemblies, parts, STLs, 2D drawings, and STEP files in Main_Model/
- Add high-resolution CAD renders, motion study, and FEA stress analysis assets in assets/
- Author comprehensive, visually rich root README.md with system architecture, hard engineering specs, and TF kinematics
- Add Main_Model/README.md with BOM, fabrication guide, and FEA simulation parameters
- Fix joint_y carriage self-collision geometry in jim.urdf.xacro
- Fix jim_sim packaging with setup.cfg (install scripts to libexec) and glob pattern in setup.py
- Update procedural field generator and SDF world with detailed boundaries and realistic crop/weed scatter
- Add one-command automated startup script (run.sh) and GitHub Actions CI workflow
- Update .gitignore and add MIT license

File: ws/src/jim_description/urdf/jim.urdf.xacro (robot description, xacro)
@@ -100,8 +100,4 @@
       <material name="jim_gold"/>
     </visual>
-    <collision>
-      <origin xyz="-0.0119 0.1865 0.0009" rpy="0 0 0"/>
-      <geometry><box size="0.042 0.415 0.062"/></geometry>
-    </collision>
   </link>
   <!-- y_carriage: Y nut, its block, laser head. -->
@@ -114,8 +110,4 @@
       <material name="jim_gold"/>
     </visual>
-    <collision>
-      <origin xyz="-0.0154 0.007 0.0093" rpy="0 0 0"/>
-      <geometry><box size="0.047 0.016 0.054"/></geometry>
-    </collision>
   </link>
   <!-- laser_aim_link: where the beam leaves the head, pointing down.
